Commit message: major bug fixes and optimization in distribution creation, fix plane urdf

File: sd_maskrcnn/data/plane/plane.urdf (robot description, URDF)
Before this commit: robot root, 1 links, 0 joints
Links:
- link link_plane_convex_piece_0: geometry collision mesh filename=plane_convex_piece_0.obj scale=1.0000E+00 1.0000E+00 1.0000E+00; visual mesh filename=plane_convex_piece_0.obj scale=1.0000E+00 1.0000E+00 1.0000E+00
